File: Projects/R0001_I3G4250D/I3G4250D_gyroscope.sch (KiCad schematic (older format))
At the start: 3 parts

Commit message: started IMU project
Parts:
- added C3, C4, C5, C6: 1uF, Capacitors_SMD:C_0805, symbol C
- added C7: 10uF tantalum, symbol C
- added C8, C9: 0.1uF, Capacitors_SMD:C_0805, symbol C
- added D1: POW, LEDs:LED-0805, symbol LED
- added J1: modular8_rev3_comms_in, Libraries - KiCAD:modular8_rev3_edge, symbol modular8_rev3_comms_in
- added J2: modular8_rev3_comms_out, Libraries - KiCAD:modular8_rev3_edge, symbol modular8_rev3_comms_out
- added LDO1, LDO2: AP7313-33SAG-7, TO_SOT_Packages_SMD:SOT-23, symbol AP7313-33SAG-7
- added R1: 10k, Resistors_SMD:R_0805, symbol R
- added R2: 680, Resistors_SMD:R_0805, symbol R
- added RP1: R_PACK4, Resistors_SMD:R_Array_Convex_4x0603, symbol R_PACK4
- added U2: ADXL343, symbol ADXL343
- C1: renamed from C?; value C -> 10nF; footprint (none) -> Capacitors_SMD:C_0805
- C2: renamed from C?; value C -> 0.47uF; footprint (none) -> Capacitors_SMD:C_0805
- gave numbers to parts that had none: 1
Connections:
- net +3V3: now reaches U1.1 (VDD_IO)
- net +3V3: now also U1.5 (CS), C6.1, C8.1, C9.1, LDO2.2 (OUT), U2.1 (VDD_IO), U2.7 (~CS)
- net GND: now reaches U1.10 (RES/GND)
- net GND: now also C1.2, U1.11 (RES/GND), U1.12 (RES/GND), U1.13 (GND), U1.4 (SDO/SA0), U1.8 (RES/GND), U1.9 (RES/GND), C3.2, C4.2, C5.2, C6.2, C7.2, C8.2, C9.2, J1.6 (GND), J1.7 (GND), J2.5 (GND), J2.8 (GND), LDO1.3 (GND), LDO2.3 (GND), R2.2, U2.11 (RES/GND), U2.12 (SDO/ALT_ADDR), U2.2 (GND), U2.3 (RES/NC), U2.4 (GND), U2.5 (GND)
- net at U1.14 (PLLFILT): now also C1.1
- net +3.3VP: now reaches U1.15 (RES/VDD)
- net +3.3VP: now also U1.16 (VDD), C5.1, C7.1, LDO1.2 (OUT), U2.6 (VDD)
- net SCL: now reaches U1.2 (SCL/SPC)
- net SCL: now also J1.12 (SCL), J2.2 (SCL), U2.14 (SCL/SCLK)
- net SDA: now reaches U1.3 (SDA/SDI/SDO)
- net SDA: now also J1.9 (SDA), J2.3 (SDA), U2.13 (SDA/SDI/SDIO)
- net U1_INT2: now reaches U1.6 (DRDY/INT2)
- net U1_INT2: now also RP1.7 (R2)
- net U1_INT1: now reaches U1.7 (INT1)
- net U1_INT1: now also RP1.8 (R1)
- net at C2.2: now also R1.1
- new net: D1.1 (K), R2.1
- new net +5V: C3.1, C4.1, D1.2 (A), J1.11 (5V), J1.2 (5V), J2.1 (5V), J2.12 (5V), LDO1.1 (IN), LDO2.1 (IN)
- new net THRU1: J1.1 (MISO), J2.11 (MISO), RP1.1 (P1)
- new net THRU2: J1.3 (SCK), J2.9 (SCK), RP1.2 (P2)
- new net THRU3: J1.5 (~RST), J2.7 (~SS), RP1.3 (P3)
- new net THRU4: J1.10 (TX/THRU), J2.4 (RX/THRU)
- new net THRU5: J1.8 (RX), J2.6 (TX)
- new net THRU6: J1.4 (MOSI), J2.10 (MOSI), RP1.4 (P4)
- new net U2_INT1: RP1.6 (R3), U2.8 (INT1)
- new net U2_INT2: RP1.5 (R4), U2.9 (INT2)
Other:
- note added: "I2C 1010011"
- note added: "I2C 1101000"
- note added: "Optional, do not populate \nif interrupts not needed"
- note added: "Place 0.1uF caps close to VDD_IO of ICs"
- moved on the sheet: C1, C2, U1
