File: Projects/R0001_I3G4250D/_saved_I3G4250D_gyroscope.sch (KiCad schematic (older format))
At the start: 19 parts, among them J1 modular8_rev3_comms_in, J2 modular8_rev3_comms_out, U1 I3G4250DTR, U2 ADXL343

Commit message: started IMU project
Parts:
- C1, C2, C3, C4, C5, C6, C8, C9: footprint (none) -> Capacitors_SMD:C_0805
- D1: footprint (none) -> LEDs:LED-0805
- J1, J2: footprint (none) -> Libraries - KiCAD:modular8_rev3_edge
- LDO1, LDO2: footprint (none) -> TO_SOT_Packages_SMD:SOT-23
- R1, R2: footprint (none) -> Resistors_SMD:R_0805
- RP1: footprint (none) -> Resistors_SMD:R_Array_Convex_4x0603
- U1: footprint (none) -> Libraries - KiCAD:LGA-16
- U2: footprint (none) -> Libraries - KiCAD:LGACC-14-1
Changed lines of the file:
@@
 F 0 "U1" H 1750 5100 60  0000 C CNN
 F 1 "I3G4250DTR" H 3250 5050 60  0000 C CNN
-F 2 "" H 2300 4450 60  0000 C CNN
+F 2 "Libraries - KiCAD:LGA-16" H 2300 4450 60  0001 C CNN
 F 3 "" H 2300 4450 60  0000 C CNN
 	1    2300 4450
@@
 F 0 "C1" V 1800 2850 50  0000 L CNN
 F 1 "10nF" V 1800 3000 50  0000 L CNN
-F 2 "" H 1988 2850 30  0000 C CNN
+F 2 "Capacitors_SMD:C_0805" H 1988 2850 30  0001 C CNN
 F 3 "" H 1950 3000 60  0000 C CNN
 	1    1950 3000
@@
 F 0 "C2" V 2050 3450 50  0000 L CNN
 F 1 "0.47uF" V 2150 3450 50  0000 L CNN
-F 2 "" H 2138 3100 30  0000 C CNN
+F 2 "Capacitors_SMD:C_0805" H 2138 3100 30  0001 C CNN
 F 3 "" H 2100 3250 60  0000 C CNN
 	1    2100 3250
@@
 F 0 "U2" H 5100 4750 60  0000 C CNN
 F 1 "ADXL343" H 6250 4750 60  0000 C CNN
-F 2 "" H 5400 4900 60  0000 C CNN
+F 2 "Libraries - KiCAD:LGACC-14-1" H 5400 4900 60  0001 C CNN
 F 3 "" H 5400 4900 60  0000 C CNN
 	1    5750 4350
@@
 F 0 "C8" H 9575 3300 50  0000 L CNN
 F 1 "0.1uF" H 9575 3100 50  0000 L CNN
-F 2 "" H 9588 3050 30  0000 C CNN
+F 2 "Capacitors_SMD:C_0805" H 9588 3050 30  0001 C CNN
 F 3 "" H 9550 3200 60  0000 C CNN
 	1    9550 3200
@@
 $EndComp
 $Comp
-L GND #PWR7
+L GND #PWR01
 U 1 1 5609AC79
 P 2900 1950
-F 0 "#PWR7" H 2900 1700 50  0001 C CNN
+F 0 "#PWR01" H 2900 1700 50  0001 C CNN
 F 1 "GND" H 2900 1800 50  0000 C CNN
 F 2 "" H 2900 1950 60  0000 C CNN
@@
 $EndComp
 $Comp
-L +3V3 #PWR23
+L +3V3 #PWR02
 U 1 1 5609ACA9
 P 9900 2850
-F 0 "#PWR23" H 9900 2700 50  0001 C CNN
+F 0 "#PWR02" H 9900 2700 50  0001 C CNN
 F 1 "+3V3" H 9900 2990 50  0000 C CNN
 F 2 "" H 9900 2850 60  0000 C CNN
@@
 F 0 "R1" V 1880 3250 50  0000 C CNN
 F 1 "10k" V 1800 3250 50  0000 C CNN
-F 2 "" V 1730 3250 30  0000 C CNN
+F 2 "Resistors_SMD:R_0805" V 1730 3250 30  0001 C CNN
 F 3 "" H 1800 3250 30  0000 C CNN
 	1    1800 3250
@@
 $EndComp
 $Comp
-L GND #PWR2
+L GND #PWR03
 U 1 1 5609B831
 P 1650 3500
-F 0 "#PWR2" H 1650 3250 50  0001 C CNN
+F 0 "#PWR03" H 1650 3250 50  0001 C CNN
 F 1 "GND" H 1650 3350 50  0000 C CNN
 F 2 "" H 1650 3500 60  0000 C CNN
@@
 I2C 1101000
 $Comp
-L GND #PWR9
+L GND #PWR04
 U 1 1 5609C139
 P 3100 4600
-F 0 "#PWR9" H 3100 4350 50  0001 C CNN
+F 0 "#PWR04" H 3100 4350 50  0001 C CNN
 F 1 "GND" H 3100 4450 50  0000 C CNN
 F 2 "" H 3100 4600 60  0000 C CNN
@@
 $EndComp
 $Comp
-L GND #PWR1
+L GND #PWR05
 U 1 1 5609C276
 P 1500 5250
-F 0 "#PWR1" H 1500 5000 50  0001 C CNN
+F 0 "#PWR05" H 1500 5000 50  0001 C CNN
 F 1 "GND" H 1500 5100 50  0000 C CNN
 F 2 "" H 1500 5250 60  0000 C CNN
@@
 F 0 "J1" H 4300 2400 60  0000 C CNN
 F 1 "modular8_rev3_comms_in" H 4000 2300 60  0000 C CNN
-F 2 "" H 3950 1900 60  0000 C CNN
+F 2 "Libraries - KiCAD:modular8_rev3_edge" H 3950 1900 60  0001 C CNN
 F 3 "" H 3950 1900 60  0000 C CNN
 	1    3950 1900
@@
 F 0 "J2" H 4300 6700 60  0000 C CNN
 F 1 "modular8_rev3_comms_out" H 3950 6600 60  0000 C CNN
-F 2 "" H 3950 6200 60  0000 C CNN
+F 2 "Libraries - KiCAD:modular8_rev3_edge" H 3950 6200 60  0001 C CNN
 F 3 "" H 3950 6200 60  0000 C CNN
 	1    3950 6200
@@
 $EndComp
 $Comp
-L +5V #PWR5
+L +5V #PWR06
 U 1 1 560B73B9
 P 2850 5950
-F 0 "#PWR5" H 2850 5800 50  0001 C CNN
+F 0 "#PWR06" H 2850 5800 50  0001 C CNN
 F 1 "+5V" H 2850 6090 50  0000 C CNN
 F 2 "" H 2850 5950 60  0000 C CNN
@@
 $EndComp
 $Comp
-L +5V #PWR11
+L +5V #PWR07
 U 1 1 560B73F4
 P 4550 6450
-F 0 "#PWR11" H 4550 6300 50  0001 C CNN
+F 0 "#PWR07" H 4550 6300 50  0001 C CNN
 F 1 "+5V" H 4550 6590 50  0000 C CNN
 F 2 "" H 4550 6450 60  0000 C CNN
@@
 $EndComp
 $Comp
-L +5V #PWR13
+L +5V #PWR08
 U 1 1 560B7533
 P 5150 1650
-F 0 "#PWR13" H 5150 1500 50  0001 C CNN
+F 0 "#PWR08" H 5150 1500 50  0001 C CNN
 F 1 "+5V" H 5150 1790 50  0000 C CNN
 F 2 "" H 5150 1650 60  0000 C CNN
@@
 $EndComp
 $Comp
-L +5V #PWR10
+L +5V #PWR09
 U 1 1 560B75BC
 P 3350 2150
-F 0 "#PWR10" H 3350 2000 50  0001 C CNN
+F 0 "#PWR09" H 3350 2000 50  0001 C CNN
 F 1 "+5V" H 3350 2290 50  0000 C CNN
 F 2 "" H 3350 2150 60  0000 C CNN
@@
 $EndComp
 $Comp
-L GND #PWR15
+L GND #PWR010
 U 1 1 560B7720
 P 5200 6450
-F 0 "#PWR15" H 5200 6200 50  0001 C CNN
+F 0 "#PWR010" H 5200 6200 50  0001 C CNN
 F 1 "GND" H 5200 6300 50  0000 C CNN
 F 2 "" H 5200 6450 60  0000 C CNN
@@
 $EndComp
 $Comp
-L GND #PWR6
+L GND #PWR011
 U 1 1 560B7752
 P 2850 6150
-F 0 "#PWR6" H 2850 5900 50  0001 C CNN
+F 0 "#PWR011" H 2850 5900 50  0001 C CNN
 F 1 "GND" H 2850 6000 50  0000 C CNN
 F 2 "" H 2850 6150 60  0000 C CNN
@@
 $EndComp
 $Comp
-L GND #PWR14
+L GND #PWR012
 U 1 1 560B7784
 P 5150 1850
-F 0 "#PWR14" H 5150 1600 50  0001 C CNN
+F 0 "#PWR012" H 5150 1600 50  0001 C CNN
 F 1 "GND" H 5150 1700 50  0000 C CNN
 F 2 "" H 5150 1850 60  0000 C CNN
@@
 SCL
 $Comp
-L +3V3 #PWR8
+L +3V3 #PWR013
 U 1 1 560B90B1
 P 3100 4300
-F 0 "#PWR8" H 3100 4150 50  0001 C CNN
+F 0 "#PWR013" H 3100 4150 50  0001 C CNN
 F 1 "+3V3" H 3100 4440 50  0000 C CNN
 F 2 "" H 3100 4300 60  0000 C CNN
@@
 $EndComp
 $Comp
-L +3.3VP #PWR3
+L +3.3VP #PWR014
 U 1 1 560B9221
 P 2450 3550
-F 0 "#PWR3" H 2600 3500 50  0001 C CNN
+F 0 "#PWR014" H 2600 3500 50  0001 C CNN
 F 1 "+3.3VP" H 2450 3650 50  0000 C CNN
 F 2 "" H 2450 3550 60  0000 C CNN
@@
 $EndComp
 $Comp
-L +3V3 #PWR17
+L +3V3 #PWR015
 U 1 1 560B92F6
 P 6650 4100
-F 0 "#PWR17" H 6650 3950 50  0001 C CNN
+F 0 "#PWR015" H 6650 3950 50  0001 C CNN
 F 1 "+3V3" H 6650 4240 50  0000 C CNN
 F 2 "" H 6650 4100 60  0000 C CNN
@@
 $EndComp
 $Comp
-L +3.3VP #PWR18
+L +3.3VP #PWR016
 U 1 1 560B96E7
 P 6650 4650
-F 0 "#PWR18" H 6800 4600 50  0001 C CNN
+F 0 "#PWR016" H 6800 4600 50  0001 C CNN
 F 1 "+3.3VP" H 6650 4750 50  0000 C CNN
 F 2 "" H 6650 4650 60  0000 C CNN
@@
 $EndComp
 $Comp
-L +3V3 #PWR16
+L +3V3 #PWR017
 U 1 1 560B9BA1
 P 5750 4900
-F 0 "#PWR16" H 5750 4750 50  0001 C CNN
+F 0 "#PWR017" H 5750 4750 50  0001 C CNN
 F 1 "+3V3" H 5750 5040 50  0000 C CNN
 F 2 "" H 5750 4900 60  0000 C CNN
@@
 $EndComp
 $Comp
-L +3V3 #PWR4
+L +3V3 #PWR018
 U 1 1 560B9BF7
 P 2450 5250
-F 0 "#PWR4" H 2450 5100 50  0001 C CNN
+F 0 "#PWR018" H 2450 5100 50  0001 C CNN
 F 1 "+3V3" H 2450 5390 50  0000 C CNN
 F 2 "" H 2450 5250 60  0000 C CNN
@@
 $EndComp
 $Comp
-L GND #PWR19
+L GND #PWR019
 U 1 1 560B9C29
 P 6900 4500
-F 0 "#PWR19" H 6900 4250 50  0001 C CNN
+F 0 "#PWR019" H 6900 4250 50  0001 C CNN
 F 1 "GND" H 6900 4350 50  0000 C CNN
 F 2 "" H 6900 4500 60  0000 C CNN
@@
 $EndComp
 $Comp
-L GND #PWR12
+L GND #PWR020
 U 1 1 560B9E1D
 P 4600 4200
-F 0 "#PWR12" H 4600 3950 50  0001 C CNN
+F 0 "#PWR020" H 4600 3950 50  0001 C CNN
 F 1 "GND" H 4600 4050 50  0000 C CNN
 F 2 "" H 4600 4200 60  0000 C CNN
@@
 F 0 "LDO2" H 8800 3200 60  0000 C CNN
 F 1 "AP7313-33SAG-7" H 8600 3100 60  0000 C CNN
-F 2 "" H 8600 2950 60  0000 C CNN
+F 2 "TO_SOT_Packages_SMD:SOT-23" H 8600 2950 60  0001 C CNN
 F 3 "" H 8600 2950 60  0000 C CNN
 	1    8600 2950
@@
 F 0 "LDO1" H 8800 2300 60  0000 C CNN
 F 1 "AP7313-33SAG-7" H 8600 2200 60  0000 C CNN
-F 2 "" H 8600 2050 60  0000 C CNN
+F 2 "TO_SOT_Packages_SMD:SOT-23" H 8600 2050 60  0001 C CNN
 F 3 "" H 8600 2050 60  0000 C CNN
 	1    8600 2050
@@
 $EndComp
 $Comp
-L +5V #PWR20
+L +5V #PWR021
 U 1 1 560BAA7D
 P 7650 1950
-F 0 "#PWR20" H 7650 1800 50  0001 C CNN
+F 0 "#PWR021" H 7650 1800 50  0001 C CNN
 F 1 "+5V" H 7650 2090 50  0000 C CNN
 F 2 "" H 7650 1950 60  0000 C CNN
@@
 F 0 "C4" H 7975 2400 50  0000 L CNN
 F 1 "1uF" H 7975 2200 50  0000 L CNN
-F 2 "" H 7988 2150 30  0000 C CNN
+F 2 "Capacitors_SMD:C_0805" H 7988 2150 30  0001 C CNN
 F 3 "" H 7950 2300 60  0000 C CNN
 	1    7950 2300
@@
 F 0 "C3" H 7675 3300 50  0000 L CNN
 F 1 "1uF" H 7675 3100 50  0000 L CNN
-F 2 "" H 7688 3050 30  0000 C CNN
+F 2 "Capacitors_SMD:C_0805" H 7688 3050 30  0001 C CNN
 F 3 "" H 7650 3200 60  0000 C CNN
 	1    7650 3200
@@
 F 0 "C5" H 9225 2400 50  0000 L CNN
 F 1 "1uF" H 9225 2200 50  0000 L CNN
-F 2 "" H 9238 2150 30  0000 C CNN
+F 2 "Capacitors_SMD:C_0805" H 9238 2150 30  0001 C CNN
 F 3 "" H 9200 2300 60  0000 C CNN
 	1    9200 2300
@@
 F 0 "C6" H 9225 3300 50  0000 L CNN
 F 1 "1uF" H 9225 3100 50  0000 L CNN
-F 2 "" H 9238 3050 30  0000 C CNN
+F 2 "Capacitors_SMD:C_0805" H 9238 3050 30  0001 C CNN
 F 3 "" H 9200 3200 60  0000 C CNN
 	1    9200 3200
@@
 F 0 "C7" H 9575 2400 50  0000 L CNN
 F 1 "10uF tantalum" H 9575 2200 50  0000 L CNN
-F 2 "" H 9588 2150 30  0000 C CNN
+F 2 "" H 9588 2150 30  0001 C CNN
 F 3 "" H 9550 2300 60  0000 C CNN
 	1    9550 2300
@@
 F 0 "C9" H 9925 3300 50  0000 L CNN
 F 1 "0.1uF" H 9925 3100 50  0000 L CNN
-F 2 "" H 9938 3050 30  0000 C CNN
+F 2 "Capacitors_SMD:C_0805" H 9938 3050 30  0001 C CNN
 F 3 "" H 9900 3200 60  0000 C CNN
 	1    9900 3200
@@
 $EndComp
 $Comp
-L +3.3VP #PWR22
+L +3.3VP #PWR022
 U 1 1 560BC231
 P 9550 1900
-F 0 "#PWR22" H 9700 1850 50  0001 C CNN
+F 0 "#PWR022" H 9700 1850 50  0001 C CNN
 F 1 "+3.3VP" H 9550 2000 50  0000 C CNN
 F 2 "" H 9550 1900 60  0000 C CNN
@@
 Connection ~ 9550 3450
 $Comp
-L GND #PWR21
+L GND #PWR023
 U 1 1 560BC7D1
 P 7650 3600
-F 0 "#PWR21" H 7650 3350 50  0001 C CNN
+F 0 "#PWR023" H 7650 3350 50  0001 C CNN
 F 1 "GND" H 7650 3450 50  0000 C CNN
 F 2 "" H 7650 3600 60  0000 C CNN
@@
 F 0 "RP1" H 7750 6200 50  0000 C CNN
 F 1 "R_PACK4" H 7750 5700 50  0000 C CNN
-F 2 "" H 7750 5750 60  0000 C CNN
+F 2 "Resistors_SMD:R_Array_Convex_4x0603" H 7750 5750 60  0001 C CNN
 F 3 "" H 7750 5750 60  0000 C CNN
 	1    7750 5750
@@
 F 0 "R2" V 7430 2850 50  0000 C CNN
 F 1 "680" V 7350 2850 50  0000 C CNN
-F 2 "" V 7280 2850 30  0000 C CNN
+F 2 "Resistors_SMD:R_0805" V 7280 2850 30  0001 C CNN
 F 3 "" H 7350 2850 30  0000 C CNN
 	1    7350 2850
@@
 F 0 "D1" V 7350 2550 50  0000 C CNN
 F 1 "POW" V 7350 2250 50  0000 C CNN
-F 2 "" H 7350 2400 60  0000 C CNN
+F 2 "LEDs:LED-0805" H 7350 2400 60  0001 C CNN
 F 3 "" H 7350 2400 60  0000 C CNN
 	1    7350 2400
