File: Projects/P0002_modular8/modular8_rev3.kicad_pcb (KiCad board)
At the start: 4 copper layers, 30.5 x 30.5 mm, 27 parts, among them IC1 ATMEGA328P-M, J1 modular8_rev3_comms_out, J2 modular8_rev3_comms_in, J3 modular8_rev3_interface_master, J4 modular8_rev3_interface_master, U1 LM4040D20IDBZR

Commit message: Added extra silkscreen info, README
Other:
- board text added: "2.048V Aref"
- board text added: "3.3V in/outputs"
- board text added: "modular8.com/0002"
- board text removed: "modular8.com/006"
Changed lines of the file:
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@@
     (links 84)
     (no_connects 0)
-    (area 117.337666 97.881 162.062335 130.569)
+    (area 117.337666 98.984999 163.061954 134.594601)
     (thickness 1.6)
-    (drawings 71)
+    (drawings 76)
     (tracks 461)
     (zones 0)
@@
   (page A4)
   (layers
-    (0 F.Cu signal)
-    (1 In1.Cu power)
-    (2 In2.Cu signal)
+    (0 F.Cu signal hide)
+    (1 In1.Cu power hide)
+    (2 In2.Cu signal hide)
     (31 B.Cu signal)
     (32 B.Adhes user hide)
@@
     (34 B.Paste user)
     (35 F.Paste user hide)
-    (36 B.SilkS user hide)
-    (37 F.SilkS user)
+    (36 B.SilkS user)
+    (37 F.SilkS user hide)
     (38 B.Mask user)
     (39 F.Mask user)
@@
     (visible_elements 7FFE7FFF)
     (pcbplotparams
-      (layerselection 0x00030_80000001)
+      (layerselection 0x011f8_80000007)
       (usegerberextensions false)
       (excludeedgelayer true)
@@
       (psa4output false)
       (plotreference true)
-      (plotvalue true)
+      (plotvalue false)
       (plotinvisibletext false)
       (padsonsilk false)
@@
       (drillshape 0)
       (scaleselection 1)
-      (outputdirectory ""))
+      (outputdirectory Gerbers/))
   )
   (net 0 "")
@@
     )
   )
+  (dimension 25.4 (width 0.1524) (layer Dwgs.User)
+    (gr_text "1.0000 in" (at 139.7 133.9723) (layer Dwgs.User)
+      (effects (font (size 0.635 0.635) (thickness 0.1524)))
+    )
+    (feature1 (pts (xy 152.4 127) (xy 152.4 134.5946)))
+    (feature2 (pts (xy 127 127) (xy 127 134.5946)))
+    (crossbar (pts (xy 127 133.35) (xy 152.4 133.35)))
+    (arrow1a (pts (xy 152.4 133.35) (xy 151.273496 133.936421)))
+    (arrow1b (pts (xy 152.4 133.35) (xy 151.273496 132.763579)))
+    (arrow2a (pts (xy 127 133.35) (xy 128.126504 133.936421)))
+    (arrow2b (pts (xy 127 133.35) (xy 128.126504 132.763579)))
+  )
+  (dimension 6.35 (width 0.1524) (layer Dwgs.User)
+    (gr_text "0.2500 in" (at 160.6423 126.365 90) (layer Dwgs.User)
+      (effects (font (size 0.635 0.635) (thickness 0.1524)))
+    )
+    (feature1 (pts (xy 154.94 123.19) (xy 161.2646 123.19)))
+    (feature2 (pts (xy 154.94 129.54) (xy 161.2646 129.54)))
+    (crossbar (pts (xy 160.02 129.54) (xy 160.02 123.19)))
+    (arrow1a (pts (xy 160.02 123.19) (xy 160.606421 124.316504)))
+    (arrow1b (pts (xy 160.02 123.19) (xy 159.433579 124.316504)))
+    (arrow2a (pts (xy 160.02 129.54) (xy 160.606421 128.413496)))
+    (arrow2b (pts (xy 160.02 129.54) (xy 159.433579 128.413496)))
+  )
+  (dimension 17.78 (width 0.1524) (layer Dwgs.User)
+    (gr_text "0.7000 in" (at 158.1023 114.3 90) (layer Dwgs.User)
+      (effects (font (size 0.635 0.635) (thickness 0.1524)))
+    )
+    (feature1 (pts (xy 154.94 105.41) (xy 158.7246 105.41)))
+    (feature2 (pts (xy 154.94 123.19) (xy 158.7246 123.19)))
+    (crossbar (pts (xy 157.48 123.19) (xy 157.48 105.41)))
+    (arrow1a (pts (xy 157.48 105.41) (xy 158.066421 106.536504)))
+    (arrow1b (pts (xy 157.48 105.41) (xy 156.893579 106.536504)))
+    (arrow2a (pts (xy 157.48 123.19) (xy 158.066421 122.063496)))
+    (arrow2b (pts (xy 157.48 123.19) (xy 156.893579 122.063496)))
+  )
+  (gr_text "2.048V Aref" (at 135.128 122.174) (layer F.SilkS)
+    (effects (font (size 0.635 0.635) (thickness 0.1524)))
+  )
+  (gr_text "3.3V in/outputs" (at 136.144 121.158) (layer F.SilkS)
+    (effects (font (size 0.635 0.635) (thickness 0.1524)))
+  )
   (gr_text "Max Prokopenko" (at 145.415 109.855) (layer B.SilkS)
     (effects (font (size 0.635 0.635) (thickness 0.1524)) (justify mirror))
   )
-  (gr_text openrobotics.ca (at 139.446 121.666) (layer B.SilkS)
-    (effects (font (size 1.27 1.27) (thickness 0.1524)) (justify mirror))
-  )
-  (gr_text modular8.com/006 (at 140.208 106.934) (layer B.SilkS)
-    (effects (font (size 1.27 1.27) (thickness 0.1524)) (justify mirror))
+  (gr_text openrobotics.ca (at 138.43 121.92) (layer B.SilkS)
+    (effects (font (size 1.016 1.016) (thickness 0.1524)) (justify mirror))
+  )
+  (gr_text modular8.com/0002 (at 140.208 106.934) (layer B.SilkS)
+    (effects (font (size 1.016 1.016) (thickness 0.1524)) (justify mirror))
   )
   (gr_text SCL (at 144.78 103.378 270) (layer B.SilkS)
