File: Projects/P0002_modular8/modular8_rev3.kicad_pcb (KiCad board)
At the start: 4 copper layers, 30.5 x 30.5 mm, 27 parts, among them IC1 ATMEGA328P-M, J1 modular8_rev3_comms_out, J2 modular8_rev3_comms_in, J3 modular8_rev3_interface_master, J4 modular8_rev3_interface_master, U1 LM4040D20IDBZR

Commit message: Updated module rev3
Routing:
- net (no net): track 0.00 -> 0.96 mm, vias 0 -> 2
Changed lines of the file:
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@@
-(kicad_pcb (version 4) (host pcbnew 4.0.0-rc1-stable)
+(kicad_pcb (version 4) (host pcbnew 4.0.1-stable)
   (general
-    (links 84)
+    (links 0)
     (no_connects 0)
     (area 117.337666 98.984999 163.061954 134.594601)
     (thickness 1.6)
     (drawings 76)
-    (tracks 461)
+    (tracks 474)
     (zones 0)
     (modules 27)
@@
     (pcbplotparams
       (layerselection 0x011f8_80000007)
-      (usegerberextensions false)
+      (usegerberextensions true)
       (excludeedgelayer true)
       (linewidth 0.100000)
@@
   (gr_line (start 154.94 123.19) (end 154.94 129.54) (angle 90) (layer Edge.Cuts) (width 0.15))
   (gr_line (start 152.4 123.19) (end 154.94 123.19) (angle 90) (layer Edge.Cuts) (width 0.15))
+  (segment (start 138.8375 113.4375) (end 138.45539 113.4375) (width 0.1524) (layer F.Cu) (net 0))
+  (via (at 138.45539 113.4375) (size 0.508) (drill 0.3302) (layers F.Cu B.Cu) (net 0))
+  (segment (start 138.849275 115.1625) (end 138.992917 115.306142) (width 0.1524) (layer F.Cu) (net 0))
+  (segment (start 138.8375 115.1625) (end 138.849275 115.1625) (width 0.1524) (layer F.Cu) (net 0))
+  (via (at 138.992917 115.665352) (size 0.508) (drill 0.3302) (layers F.Cu B.Cu) (net 0))
+  (segment (start 138.992917 115.306142) (end 138.992917 115.665352) (width 0.1524) (layer F.Cu) (net 0))
   (segment (start 135.3248 116.205) (end 135.128 116.205) (width 0.3048) (layer F.Cu) (net 1))
   (segment (start 135.636 116.5162) (end 135.3248 116.205) (width 0.3048) (layer F.Cu) (net 1))
@@
   (segment (start 128.27 110.49) (end 129.6924 110.49) (width 0.1524) (layer B.Cu) (net 16))
   (segment (start 129.6924 110.49) (end 129.9464 110.236) (width 0.1524) (layer B.Cu) (net 16))
+  (segment (start 129.9464 110.236) (end 136.017 110.236) (width 0.1524) (layer B.Cu) (net 16))
+  (segment (start 139.446 118.00479) (end 139.446 118.364) (width 0.1524) (layer B.Cu) (net 16))
   (segment (start 136.017 110.236) (end 139.446 113.665) (width 0.1524) (layer B.Cu) (net 16))
-  (segment (start 129.9464 110.236) (end 136.017 110.236) (width 0.1524) (layer B.Cu) (net 16))
-  (segment (start 139.446 113.665) (end 139.446 118.00479) (width 0.1524) (layer B.Cu) (net 16))
-  (segment (start 139.446 118.00479) (end 139.446 118.364) (width 0.1524) (layer B.Cu) (net 16))
+  (segment (start 139.446 113.665) (end 139.446 115.30684) (width 0.1524) (layer B.Cu) (net 16))
+  (segment (start 139.446 115.30684) (end 139.7508 115.61164) (width 0.1524) (layer B.Cu) (net 16))
+  (segment (start 139.7508 115.61164) (end 139.7508 116.275536) (width 0.1524) (layer B.Cu) (net 16))
+  (segment (start 139.7508 116.275536) (end 139.446 116.580336) (width 0.1524) (layer B.Cu) (net 16))
+  (segment (start 139.446 116.580336) (end 139.446 118.00479) (width 0.1524) (layer B.Cu) (net 16))
   (segment (start 139.446 118.364) (end 139.446 116.704) (width 0.1524) (layer F.Cu) (net 16))
   (segment (start 139.446 116.704) (end 139.45 116.7) (width 0.1524) (layer F.Cu) (net 16))
   (via (at 139.446 118.364) (size 0.508) (drill 0.3302) (layers F.Cu B.Cu) (net 16))
-  (segment (start 139.954 117.856) (end 139.954 113.665) (width 0.1524) (layer B.Cu) (net 17))
-  (segment (start 139.954 113.665) (end 136.144 109.855) (width 0.1524) (layer B.Cu) (net 17))
-  (segment (start 136.144 109.855) (end 132.334004 109.855) (width 0.1524) (layer B.Cu) (net 17))
-  (segment (start 132.334004 109.855) (end 130.683003 108.203999) (width 0.1524) (layer B.Cu) (net 17))
-  (segment (start 130.683003 108.203999) (end 130.429004 107.95) (width 0.1524) (layer B.Cu) (net 17))
+  (segment (start 139.954 117.49679) (end 140.15591 117.29488) (width 0.1524) (layer B.Cu) (net 17))
+  (segment (start 139.954 117.856) (end 139.954 117.49679) (width 0.1524) (layer B.Cu) (net 17))
+  (segment (start 139.954 115.383774) (end 139.954 113.665) (width 0.1524) (layer B.Cu) (net 17))
+  (segment (start 140.15591 117.29488) (end 140.15591 115.585683) (width 0.1524) (layer B.Cu) (net 17))
+  (segment (start 140.15591 115.585683) (end 139.954 115.383774) (width 0.1524) (layer B.Cu) (net 17))
+  (segment (start 139.954 113.665) (end 134.239 107.95) (width 0.1524) (layer B.Cu) (net 17))
+  (segment (start 134.239 107.95) (end 130.788214 107.95) (width 0.1524) (layer B.Cu) (net 17))
+  (segment (start 130.788214 107.95) (end 130.429004 107.95) (width 0.1524) (layer B.Cu) (net 17))
   (segment (start 128.27 107.95) (end 130.429004 107.95) (width 0.1524) (layer F.Cu) (net 17))
   (via (at 130.429004 107.95) (size 0.508) (drill 0.3302) (layers F.Cu B.Cu) (net 17))
@@
   (segment (start 135.89 105.283) (end 135.89 102.87) (width 0.1524) (layer B.Cu) (net 33))
   (segment (start 140.486 106.934) (end 140.486 106.734) (width 0.1524) (layer F.Cu) (net 33))
+  (segment (start 138.938 114.939392) (end 138.176 115.701392) (width 0.1524) (layer In2.Cu) (net 35))
+  (segment (start 138.176 119.126) (end 141.986001 122.936001) (width 0.1524) (layer In2.Cu) (net 35))
+  (segment (start 138.938 108.712) (end 138.938 114.939392) (width 0.1524) (layer In2.Cu) (net 35))
+  (segment (start 141.986001 122.936001) (end 142.24 123.19) (width 0.1524) (layer In2.Cu) (net 35))
+  (segment (start 138.176 115.701392) (end 138.176 119.126) (width 0.1524) (layer In2.Cu) (net 35))
   (segment (start 143.51 125.73) (end 143.51 124.46) (width 0.1524) (layer B.Cu) (net 35))
   (segment (start 143.51 124.46) (end 142.24 123.19) (width 0.1524) (layer B.Cu) (net 35))
-  (segment (start 141.986001 122.936001) (end 142.24 123.19) (width 0.1524) (layer In2.Cu) (net 35))
-  (segment (start 138.176 119.126) (end 141.986001 122.936001) (width 0.1524) (layer In2.Cu) (net 35))
-  (segment (start 138.176 115.824) (end 138.176 119.126) (width 0.1524) (layer In2.Cu) (net 35))
-  (segment (start 138.938 115.062) (end 138.176 115.824) (width 0.1524) (layer In2.Cu) (net 35))
-  (segment (start 138.938 108.712) (end 138.938 115.062) (width 0.1524) (layer In2.Cu) (net 35))
   (via (at 142.24 123.19) (size 0.508) (drill 0.3302) (layers F.Cu B.Cu) (net 35))
   (segment (start 138.95 111.9) (end 138.95 111.3976) (width 0.1524) (layer F.Cu) (net 35))
