File: Training/T0004-5-6/usb_adapter.sch (KiCad schematic (older format))
At the start: 23 parts, among them J1 modular8_rev3_comms_out, P1 USB_OTG, U1 FT231X, U2 TE_1825058-1

Commit message: uploading initial design
Parts:
- J1: footprint (none) -> open_robotics:modular8_rev3_edge
- U2: footprint (none) -> open_robotics:DIPSWITCH_SMT_ALCO_2CCT
Changed lines of the file:
@@
 LIBS:atmel
 LIBS:contrib
+LIBS:open_robotics
 LIBS:valves
-LIBS:open_robotics
 LIBS:usb_adapter-cache
 EELAYER 25 0
@@
 $EndComp
 $Comp
-L GND #PWR1
+L GND #PWR01
 U 1 1 5622C099
 P 1850 4350
-F 0 "#PWR1" H 1850 4100 50  0001 C CNN
+F 0 "#PWR01" H 1850 4100 50  0001 C CNN
 F 1 "GND" H 1850 4200 50  0000 C CNN
 F 2 "" H 1850 4350 60  0000 C CNN
@@
 $EndComp
 $Comp
-L +5V #PWR2
+L +5V #PWR02
 U 1 1 5622C0D5
 P 2100 2600
-F 0 "#PWR2" H 2100 2450 50  0001 C CNN
+F 0 "#PWR02" H 2100 2450 50  0001 C CNN
 F 1 "+5V" H 2100 2740 50  0000 C CNN
 F 2 "" H 2100 2600 60  0000 C CNN
@@
 $EndComp
 $Comp
-L +3V3 #PWR5
+L +3V3 #PWR03
 U 1 1 5622C14E
 P 3350 3250
-F 0 "#PWR5" H 3350 3100 50  0001 C CNN
+F 0 "#PWR03" H 3350 3100 50  0001 C CNN
 F 1 "+3V3" H 3350 3390 50  0000 C CNN
 F 2 "" H 3350 3250 60  0000 C CNN
@@
 $EndComp
 $Comp
-L GND #PWR7
+L GND #PWR04
 U 1 1 5622DDA1
 P 4050 4850
-F 0 "#PWR7" H 4050 4600 50  0001 C CNN
+F 0 "#PWR04" H 4050 4600 50  0001 C CNN
 F 1 "GND" H 4050 4700 50  0000 C CNN
 F 2 "" H 4050 4850 60  0000 C CNN
@@
 $EndComp
 $Comp
-L +5V #PWR8
+L +5V #PWR05
 U 1 1 5622EF00
 P 4100 2950
-F 0 "#PWR8" H 4100 2800 50  0001 C CNN
+F 0 "#PWR05" H 4100 2800 50  0001 C CNN
 F 1 "+5V" H 4100 3090 50  0000 C CNN
 F 2 "" H 4100 2950 60  0000 C CNN
@@
 $EndComp
 $Comp
-L +3V3 #PWR9
+L +3V3 #PWR06
 U 1 1 5622F2DF
 P 4300 2950
-F 0 "#PWR9" H 4300 2800 50  0001 C CNN
+F 0 "#PWR06" H 4300 2800 50  0001 C CNN
 F 1 "+3V3" H 4300 3090 50  0000 C CNN
 F 2 "" H 4300 2950 60  0000 C CNN
@@
 ~SLEEP
 $Comp
-L +5V #PWR3
+L +5V #PWR07
 U 1 1 562300CF
 P 3300 1200
-F 0 "#PWR3" H 3300 1050 50  0001 C CNN
+F 0 "#PWR07" H 3300 1050 50  0001 C CNN
 F 1 "+5V" H 3300 1340 50  0000 C CNN
 F 2 "" H 3300 1200 60  0000 C CNN
@@
 $EndComp
 $Comp
-L +3V3 #PWR6
+L +3V3 #PWR08
 U 1 1 562301B6
 P 3850 1200
-F 0 "#PWR6" H 3850 1050 50  0001 C CNN
+F 0 "#PWR08" H 3850 1050 50  0001 C CNN
 F 1 "+3V3" H 3850 1340 50  0000 C CNN
 F 2 "" H 3850 1200 60  0000 C CNN
@@
 $EndComp
 $Comp
-L GND #PWR4
+L GND #PWR09
 U 1 1 56230399
 P 3650 1900
-F 0 "#PWR4" H 3650 1650 50  0001 C CNN
+F 0 "#PWR09" H 3650 1650 50  0001 C CNN
 F 1 "GND" H 3650 1750 50  0000 C CNN
 F 2 "" H 3650 1900 60  0000 C CNN
@@
 $EndComp
 $Comp
-L GND #PWR10
+L GND #PWR010
 U 1 1 56231F36
 P 5200 2900
-F 0 "#PWR10" H 5200 2650 50  0001 C CNN
+F 0 "#PWR010" H 5200 2650 50  0001 C CNN
 F 1 "GND" H 5200 2750 50  0000 C CNN
 F 2 "" H 5200 2900 60  0000 C CNN
@@
 $EndComp
 $Comp
-L +3V3 #PWR11
+L +3V3 #PWR011
 U 1 1 562364F3
 P 5500 1700
-F 0 "#PWR11" H 5500 1550 50  0001 C CNN
+F 0 "#PWR011" H 5500 1550 50  0001 C CNN
 F 1 "+3V3" H 5500 1840 50  0000 C CNN
 F 2 "" H 5500 1700 60  0000 C CNN
@@
 F 0 "U2" V 6850 2650 60  0000 C CNN
 F 1 "TE_1825058-1" V 6950 2900 60  0000 C CNN
-F 2 "" H 7010 2400 60  0000 C CNN
+F 2 "open_robotics:DIPSWITCH_SMT_ALCO_2CCT" H 7010 2400 60  0001 C CNN
 F 3 "" H 7010 2400 60  0000 C CNN
 	1    6900 2400
@@
 F 0 "U2" H 8900 3800 60  0000 C CNN
 F 1 "TE_1825058-1" H 9150 3700 60  0000 C CNN
-F 2 "" H 9210 3550 60  0000 C CNN
+F 2 "open_robotics:DIPSWITCH_SMT_ALCO_2CCT" H 9210 3550 60  0001 C CNN
 F 3 "" H 9210 3550 60  0000 C CNN
 	2    9100 3550
@@
 F 0 "J1" H 8250 4000 60  0000 C CNN
 F 1 "modular8_rev3_comms_out" H 7950 3900 60  0000 C CNN
-F 2 "" H 7900 3500 60  0000 C CNN
+F 2 "open_robotics:modular8_rev3_edge" H 7900 3500 60  0001 C CNN
 F 3 "" H 7900 3500 60  0000 C CNN
 	1    7900 3500
@@
 $EndComp
 $Comp
-L +5V #PWR12
+L +5V #PWR012
 U 1 1 5629BADF
 P 6900 2000
-F 0 "#PWR12" H 6900 1850 50  0001 C CNN
+F 0 "#PWR012" H 6900 1850 50  0001 C CNN
 F 1 "+5V" H 6900 2140 50  0000 C CNN
 F 2 "" H 6900 2000 60  0000 C CNN
@@
 Capacitors, resistors and ferrite bead 0603 SMT packages\nLEDs 0805 package
 $Comp
-L GND #PWR?
+L GND #PWR013
 U 1 1 562A3E08
 P 7100 3550
-F 0 "#PWR?" H 7100 3300 50  0001 C CNN
+F 0 "#PWR013" H 7100 3300 50  0001 C CNN
 F 1 "GND" H 7100 3400 50  0000 C CNN
 F 2 "" H 7100 3550 60  0000 C CNN
@@
 	7100 3550 7300 3550
 $Comp
-L GND #PWR?
+L GND #PWR014
 U 1 1 562A3EDA
 P 8600 3650
-F 0 "#PWR?" H 8600 3400 50  0001 C CNN
+F 0 "#PWR014" H 8600 3400 50  0001 C CNN
 F 1 "GND" H 8600 3500 50  0000 C CNN
 F 2 "" H 8600 3650 60  0000 C CNN
@@
 	8600 3450 8600 3650
 $Comp
-L +3V3 #PWR?
+L +3V3 #PWR015
 U 1 1 562A597E
 P 9700 3000
-F 0 "#PWR?" H 9700 2850 50  0001 C CNN
+F 0 "#PWR015" H 9700 2850 50  0001 C CNN
 F 1 "+3V3" H 9700 3140 50  0000 C CNN
 F 2 "" H 9700 3000 60  0000 C CNN

Commit message: max fixing footprint mistakes
Parts:
- removed U1: FT231X, Housings_DFN_QFN:QFN-20-1EP_4x4mm_Pitch0.5mm, symbol FT231X
- removed U2: TE_1825058-1, open_robotics:DIPSWITCH_SMT_ALCO_2CCT, symbol TE_1825058-1-RESCUE-usb_adapter
- added U1: FT231XQ, Housings_DFN_QFN:QFN-20-1EP_4x4mm_Pitch0.5mm, symbol FT231XQ
- added U2: TE_1825058-1, open_robotics:DIPSWITCH_SMT_ALCO_2CCT, symbol TE_1825058-1
Connections:
- wire segments 72 -> 73
Changed lines of the file:
@@
 LIBS:atmel
 LIBS:contrib
+LIBS:valves
 LIBS:open_robotics
-LIBS:valves
 LIBS:usb_adapter-cache
 EELAYER 25 0
@@
 1
 $Comp
-L FT231X U1
-U 1 1 5622A3C5
-P 4050 3600
-F 0 "U1" H 3700 4100 60  0000 C CNN
-F 1 "FT231X" H 3800 4000 60  0000 C CNN
-F 2 "Housings_DFN_QFN:QFN-20-1EP_4x4mm_Pitch0.5mm" H 4000 4100 60  0001 C CNN
-F 3 "" H 4000 4100 60  0000 C CNN
-	1    4050 3600
-	1    0    0    -1
-$EndComp
-$Comp
 L R R2
 U 1 1 5622A6B9
@@
 $EndComp
 $Comp
-L TE_1825058-1-RESCUE-usb_adapter U2
-U 1 1 5629AB3C
-P 6900 2400
-F 0 "U2" V 6850 2650 60  0000 C CNN
-F 1 "TE_1825058-1" V 6950 2900 60  0000 C CNN
-F 2 "open_robotics:DIPSWITCH_SMT_ALCO_2CCT" H 7010 2400 60  0001 C CNN
-F 3 "" H 7010 2400 60  0000 C CNN
-	1    6900 2400
-	0    1    1    0
-$EndComp
-$Comp
-L TE_1825058-1-RESCUE-usb_adapter U2
-U 2 1 5629ABC7
-P 9100 3550
-F 0 "U2" H 8900 3800 60  0000 C CNN
-F 1 "TE_1825058-1" H 9150 3700 60  0000 C CNN
-F 2 "open_robotics:DIPSWITCH_SMT_ALCO_2CCT" H 9210 3550 60  0001 C CNN
-F 3 "" H 9210 3550 60  0000 C CNN
-	2    9100 3550
-	1    0    0    -1
-$EndComp
-$Comp
-L modular8_rev3_comms_out J1
-U 1 1 5629AC49
-P 7900 3500
-F 0 "J1" H 8250 4000 60  0000 C CNN
-F 1 "modular8_rev3_comms_out" H 7950 3900 60  0000 C CNN
-F 2 "open_robotics:modular8_rev3_edge" H 7900 3500 60  0001 C CNN
-F 3 "" H 7900 3500 60  0000 C CNN
-	1    7900 3500
-	-1   0    0    -1
-$EndComp
-$Comp
 L +5V #PWR012
 U 1 1 5629BADF
@@
 	4000 4700 4000 4750
 Wire Wire Line
-	4000 4750 4100 4750
+	3900 4750 4100 4750
 Wire Wire Line
 	4100 4750 4100 4700
@@
 Text Notes 5950 1850 0    60   ~ 0
 Ensures that\ndevice is on
+$Comp
+L modular8_rev3_comms_out J1
+U 1 1 5629AC49
+P 7900 3500
+F 0 "J1" H 8250 4000 60  0000 C CNN
+F 1 "modular8_rev3_comms_out" H 7950 3900 60  0000 C CNN
+F 2 "open_robotics:modular8_rev3_edge" H 7900 3500 60  0001 C CNN
+F 3 "" H 7900 3500 60  0000 C CNN
+	1    7900 3500
+	-1   0    0    -1
+$EndComp
+$Comp
+L FT231XQ U1
+U 1 1 565D1F15
+P 4050 3600
+F 0 "U1" H 3700 4100 60  0000 C CNN
+F 1 "FT231XQ" H 3800 4000 60  0000 C CNN
+F 2 "Housings_DFN_QFN:QFN-20-1EP_4x4mm_Pitch0.5mm" H 4000 4100 60  0001 C CNN
+F 3 "" H 4000 4100 60  0000 C CNN
+	1    4050 3600
+	1    0    0    -1
+$EndComp
+Wire Wire Line
+	3900 4750 3900 4700
+Connection ~ 4000 4750
+$Comp
+L TE_1825058-1 U2
+U 1 1 565D260C
+P 6900 2400
+F 0 "U2" H 6650 2700 60  0000 C CNN
+F 1 "TE_1825058-1" H 6900 2600 60  0000 C CNN
+F 2 "open_robotics:DIPSWITCH_SMT_ALCO_2CCT" H 7010 2400 60  0001 C CNN
+F 3 "" H 7010 2400 60  0000 C CNN
+	1    6900 2400
+	0    -1   -1   0
+$EndComp
+$Comp
+L TE_1825058-1 U2
+U 2 1 565D26CD
+P 9100 3550
+F 0 "U2" H 8850 3850 60  0000 C CNN
+F 1 "TE_1825058-1" H 9100 3750 60  0000 C CNN
+F 2 "open_robotics:DIPSWITCH_SMT_ALCO_2CCT" H 9210 3550 60  0001 C CNN
+F 3 "" H 9210 3550 60  0000 C CNN
+	2    9100 3550
+	1    0    0    -1
+$EndComp
 $EndSCHEMATC
