File: Training/T0004-5-6/usb_adapter.kicad_pcb (KiCad board)
At the start: 2 copper layers, 50.8 x 25.4 mm, 23 parts, among them J1 modular8_rev3_comms_out, P1 USB_OTG, U1 FT231X, U2 TE_1825058-1

Commit message: added suggestions
Parts:
- U1: value FT231X -> FT231XQ
- moved U1 0.25 mm to (144.6, 112.7), turned to 270 degrees
Connections:
- U1 pad 1: Net-(C7-Pad1) -> /RX
- U1 pad 10: /~TXLED -> +3V3
- U1 pad 11: Net-(R2-Pad1) -> +3V3
- U1 pad 12: Net-(R1-Pad1) -> +5V
- U1 pad 13: +3V3 -> GND
- U1 pad 14: +3V3 -> /~RXLED
- U1 pad 15: +5V -> /TXDEN
- U1 pad 16: GND -> /~SLEEP
- U1 pad 17: /~RXLED -> /TX
- U1 pad 18: /TXDEN -> Net-(C7-Pad1)
- U1 pad 19: /~SLEEP -> Net-(U1-Pad19)
- U1 pad 20: /TX -> +3V3
- U1 pad 21: (no net) -> GND
- U1 pad 3: +3V3 -> GND
- U1 pad 4: /RX -> Net-(U1-Pad4)
- U1 pad 6: GND -> Net-(U1-Pad6)
- U1 pad 7: Net-(U1-Pad7) -> /~TXLED
- U1 pad 8: Net-(U1-Pad8) -> Net-(R2-Pad1)
- U1 pad 9: Net-(U1-Pad9) -> Net-(R1-Pad1)
- U2 pad 1: +5V -> /POWER_OUT
- U2 pad 2: /POWER_OUT -> Net-(J1-Pad7)
- U2 pad 3: (no net) -> /PROGRAM
- U2 pad 4: (no net) -> +5V
Routing:
- net /POWER_OUT: track 39.5 -> 15.5 mm, vias 2 -> 1
- net +5V: track 23.2 -> 12.7 mm, vias 1 -> 0
- net GND: track 87.4 -> 80.0 mm
- net +3V3: track 39.9 -> 33.2 mm
- net /TX: track 12.5 -> 8.88 mm
- net Net-(R1-Pad1): track 12.1 -> 10.0 mm
- net /~RXLED: track 4.50 -> 2.60 mm
- net Net-(C7-Pad1): track 1.79 -> 0.00 mm
- net /TXDEN: track 4.74 -> 2.97 mm
- net /~TXLED: track 8.13 -> 6.50 mm
- net /RX: track 5.73 -> 4.31 mm
- net /~SLEEP: track 4.43 -> 3.12 mm
- net Net-(R2-Pad1): track 12.4 -> 11.4 mm

Commit message: finished routing after fix
Parts:
- moved R5 2.69 mm to (142.5, 108.0)
- moved D1 2.16 mm to (141.5, 116.8), turned to 270 degrees
- moved D3 2.03 mm to (141.0, 109.8), turned to 90 degrees
- moved C6 1.48 mm to (149.4, 110.2)
- moved U1 1.32 mm to (144.9, 111.4)
- moved C3 1.27 mm to (144.0, 116.6)
- moved D2 1.23 mm to (146.1, 118.6)
- moved R4 0.79 mm to (149.4, 119.1)
- moved R8 0.25 mm to (147.8, 116.8)
Routing:
- net Net-(J1-Pad7): track 0.00 -> 36.0 mm, vias 0 -> 1
- net /POWER_OUT: track 15.5 -> 50.0 mm, vias 1 -> 3
- net /PROGRAM: track 7.11 -> 25.7 mm, vias 1 -> 2
- net +5V: track 12.7 -> 27.3 mm, vias 0 -> 3
- net GND: track 80.0 -> 93.2 mm, vias 3 -> 4
- net +3V3: track 33.2 -> 40.0 mm
- net /RX: track 4.31 -> 8.81 mm, vias 1 -> 3
- net /~TXLED: track 6.50 -> 2.01 mm
- net Net-(C7-Pad1): track 0.00 -> 3.68 mm
- net /~RXLED: track 2.60 -> 5.52 mm
- net Net-(D3-Pad2): track 4.44 -> 2.25 mm
- net /TX: track 8.88 -> 7.14 mm
- net Net-(J1-Pad11): track 0.00 -> 1.02 mm
- net /TXDEN: track 2.97 -> 3.99 mm
- net Net-(R2-Pad1): track 11.4 -> 10.7 mm
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Other:
- board size 50.8 x 25.4 mm -> 27.2 x 15.5 mm

Commit message: finished routing after fix
Routing:
- net GND: track 93.2 -> 96.3 mm
- net Net-(J1-Pad11): track 1.02 -> 0.00 mm
- net +3V3: track 40.0 -> 39.3 mm
Changed lines of the file:
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@@
     (links 54)
     (no_connects 0)
-    (area 126.095679 101.524999 187.015002 127.075001)
+    (area 126.095679 103.69957 187.015002 124.39243)
     (thickness 1.6)
     (drawings 4)
-    (tracks 313)
+    (tracks 314)
     (zones 0)
     (modules 23)
@@
   (segment (start 136.5958 112.1918) (end 136.02062 112.1918) (width 0.25) (layer F.Cu) (net 1))
   (segment (start 136.02062 112.1918) (end 134.62 112.1918) (width 0.25) (layer F.Cu) (net 1))
-  (segment (start 152.146 114.046) (end 152.146 113.284) (width 0.25) (layer F.Cu) (net 2))
-  (segment (start 152.146 113.284) (end 151.638 112.776) (width 0.25) (layer F.Cu) (net 2))
+  (segment (start 149.86 114.3) (end 150.114 114.3) (width 0.25) (layer F.Cu) (net 2))
+  (segment (start 150.114 114.3) (end 151.638 112.776) (width 0.25) (layer F.Cu) (net 2))
+  (segment (start 152.328999 114.228999) (end 149.931001 114.228999) (width 0.25) (layer B.Cu) (net 2))
+  (segment (start 149.931001 114.228999) (end 149.86 114.3) (width 0.25) (layer B.Cu) (net 2))
+  (via (at 149.86 114.3) (size 0.6) (drill 0.4) (layers F.Cu B.Cu) (net 2))
   (segment (start 153.233001 114.228999) (end 152.328999 114.228999) (width 0.25) (layer B.Cu) (net 2))
-  (segment (start 152.328999 114.228999) (end 152.146 114.046) (width 0.25) (layer B.Cu) (net 2))
-  (via (at 152.146 114.046) (size 0.6) (drill 0.4) (layers F.Cu B.Cu) (net 2))
   (segment (start 149.352 109.486) (end 149.352 108.836) (width 0.25) (layer F.Cu) (net 2))
   (segment (start 149.352 108.836) (end 148.974 108.458) (width 0.25) (layer F.Cu) (net 2))
@@
   (segment (start 137.543 113.792) (end 138.188 114.437) (width 0.25) (layer F.Cu) (net 5))
   (segment (start 138.188 114.437) (end 138.188 115.062) (width 0.25) (layer F.Cu) (net 5))
+  (segment (start 149.606 113.40101) (end 149.306001 113.701009) (width 0.25) (layer B.Cu) (net 6))
+  (segment (start 149.306001 113.701009) (end 148.934991 113.701009) (width 0.25) (layer B.Cu) (net 6))
+  (segment (start 148.934991 113.701009) (end 148.578 114.058) (width 0.25) (layer B.Cu) (net 6))
+  (segment (start 149.352 111.011) (end 149.977 111.636) (width 0.25) (layer F.Cu) (net 6))
+  (segment (start 149.977 111.636) (end 149.977 113.03001) (width 0.25) (layer F.Cu) (net 6))
+  (segment (start 149.977 113.03001) (end 149.606 113.40101) (width 0.25) (layer F.Cu) (net 6))
+  (via (at 149.606 113.40101) (size 0.6) (drill 0.4) (layers F.Cu B.Cu) (net 6))
+  (segment (start 146.882 110.369) (end 148.735 110.369) (width 0.25) (layer F.Cu) (net 6))
+  (segment (start 148.735 110.369) (end 149.352 110.986) (width 0.25) (layer F.Cu) (net 6))
   (segment (start 149.352 119.888) (end 148.058 119.888) (width 0.25) (layer B.Cu) (net 6))
   (segment (start 148.058 119.888) (end 147.308 120.638) (width 0.25) (layer B.Cu) (net 6))
-  (segment (start 149.86 114.554) (end 148.832 114.554) (width 0.25) (layer B.Cu) (net 6))
   (segment (start 148.832 114.554) (end 148.578 114.808) (width 0.25) (layer B.Cu) (net 6))
-  (segment (start 149.847 111.506) (end 149.847 114.541) (width 0.25) (layer F.Cu) (net 6))
-  (segment (start 149.847 114.541) (end 149.86 114.554) (width 0.25) (layer F.Cu) (net 6))
-  (via (at 149.86 114.554) (size 0.6) (drill 0.4) (layers F.Cu B.Cu) (net 6))
   (segment (start 149.352 110.986) (end 149.352 111.011) (width 0.25) (layer F.Cu) (net 6))
-  (segment (start 149.352 111.011) (end 149.847 111.506) (width 0.25) (layer F.Cu) (net 6))
-  (segment (start 146.882 110.369) (end 148.735 110.369) (width 0.25) (layer F.Cu) (net 6))
-  (segment (start 148.735 110.369) (end 149.352 110.986) (width 0.25) (layer F.Cu) (net 6))
   (segment (start 143.244 110.497998) (end 143.244 107.95) (width 0.25) (layer B.Cu) (net 6))
   (segment (start 143.217997 115.062) (end 143.217997 115.186999) (width 0.25) (layer B.Cu) (net 6))
@@
   (segment (start 140.97 110.81004) (end 141.02896 110.869) (width 0.25) (layer F.Cu) (net 13))
   (segment (start 141.02896 110.869) (end 142.952 110.869) (width 0.25) (layer F.Cu) (net 13))
+  (segment (start 131.572 120.904) (end 149.606 120.904) (width 0.25) (layer F.Cu) (net 14))
   (segment (start 131.064 120.396) (end 131.064 118.872) (width 0.25) (layer F.Cu) (net 14))
   (segment (start 151.638 120.396) (end 153.158 120.396) (width 0.25) (layer B.Cu) (net 14))
@@
   (via (at 149.606 107.234009) (size 0.6) (drill 0.4) (layers F.Cu B.Cu) (net 14))
   (segment (start 131.064 120.396) (end 131.572 120.904) (width 0.25) (layer F.Cu) (net 14))
-  (segment (start 131.572 120.904) (end 149.606 120.904) (width 0.25) (layer F.Cu) (net 14))
   (via (at 149.606 120.904) (size 0.6) (drill 0.4) (layers F.Cu B.Cu) (net 14))
   (segment (start 129.667 114.3) (end 129.667 117.475) (width 0.25) (layer B.Cu) (net 14))
@@
   (segment (start 132.91549 108.82901) (end 136.340313 108.82901) (width 0.25) (layer B.Cu) (net 16))
   (via (at 136.340313 108.82901) (size 0.6) (drill 0.4) (layers F.Cu B.Cu) (net 16))
-  (segment (start 151.638 120.396) (end 152.146 120.396) (width 0.25) (layer F.Cu) (net 18))
-  (segment (start 151.638 120.396) (end 151.13 120.396) (width 0.25) (layer F.Cu) (net 18))
   (segment (start 147.522974 113.055513) (end 149.971486 110.607001) (width 0.25) (layer B.Cu) (net 20))
   (segment (start 149.971486 110.607001) (end 151.266999 110.607001) (width 0.25) (layer B.Cu) (net 20))

Commit message: generated gerbers
Parts:
- removed U2: TE_1825058-1, open_robotics:DIPSWITCH_SMT_ALCO_2CCT
Other:
- board text added: "USB to serial Chris OpenRobotics.ca"
Changed lines of the file:
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@@
-(kicad_pcb (version 4) (host pcbnew 4.0.0-rc1-stable)
+(kicad_pcb (version 4) (host pcbnew 4.0.0-rc2-stable)
   (general
-    (links 54)
+    (links 50)
     (no_connects 0)
-    (area 126.095679 103.69957 187.015002 124.39243)
+    (area 126.924999 106.096999 154.253001 121.741001)
     (thickness 1.6)
-    (drawings 4)
+    (drawings 5)
     (tracks 314)
     (zones 0)
-    (modules 23)
+    (modules 22)
     (nets 34)
   )
   (page A4)
   (layers
-    (0 F.Cu signal)
+    (0 F.Cu signal hide)
     (31 B.Cu signal)
-    (32 B.Adhes user)
-    (33 F.Adhes user)
-    (34 B.Paste user)
-    (35 F.Paste user)
-    (36 B.SilkS user hide)
-    (37 F.SilkS user hide)
-    (38 B.Mask user)
-    (39 F.Mask user)
-    (40 Dwgs.User user)
-    (41 Cmts.User user)
-    (42 Eco1.User user)
-    (43 Eco2.User user)
+    (32 B.Adhes user hide)
+    (33 F.Adhes user hide)
+    (34 B.Paste user hide)
+    (35 F.Paste user hide)
+    (36 B.SilkS user)
+    (37 F.SilkS user)
+    (38 B.Mask user hide)
+    (39 F.Mask user hide)
+    (40 Dwgs.User user hide)
+    (41 Cmts.User user hide)
+    (42 Eco1.User user hide)
+    (43 Eco2.User user hide)
     (44 Edge.Cuts user)
-    (45 Margin user)
+    (45 Margin user hide)
     (46 B.CrtYd user)
     (47 F.CrtYd user hide)
@@
     (pad_to_mask_clearance 0.2)
     (aux_axis_origin 0 0)
-    (visible_elements 7FFFFFFF)
+    (visible_elements 7FFFF9FF)
     (pcbplotparams
-      (layerselection 0x00030_80000001)
-      (usegerberextensions false)
+      (layerselection 0x010f0_80000001)
+      (usegerberextensions true)
       (excludeedgelayer true)
       (linewidth 0.100000)
@@
       (outputformat 1)
       (mirror false)
-      (drillshape 1)
+      (drillshape 0)
       (scaleselection 1)
-      (outputdirectory ""))
+      (outputdirectory ../gerbers/Chris/))
   )
   (net 0 "")
@@
     (add_net "Net-(U1-Pad6)")
   )
+  (module Capacitors_SMD:C_0603 (layer F.Cu)
+    (at 138.696 108.458)
+    (descr "Capacitor SMD 0603, reflow soldering, AVX (see smccp.pdf)")
+    (tags "capacitor 0603")
+    (attr smd)
+    (fp_text reference C5 (at 0 -1.9) (layer F.SilkS)
+      (effects (font (size 1 1) (thickness 0.15)))
+    )
+    (fp_text value 0.1uF (at 0 1.9) (layer F.Fab)
+      (effects (font (size 1 1) (thickness 0.15)))
+    )
+    (fp_line (start -1.45 -0.75) (end 1.45 -0.75) (layer F.CrtYd) (width 0.05))
+    (fp_line (start -1.45 0.75) (end 1.45 0.75) (layer F.CrtYd) (width 0.05))
+    (fp_line (start -1.45 -0.75) (end -1.45 0.75) (layer F.CrtYd) (width 0.05))
+    (fp_line (start 1.45 -0.75) (end 1.45 0.75) (layer F.CrtYd) (width 0.05))
+    (fp_line (start -0.35 -0.6) (end 0.35 -0.6) (layer F.SilkS) (width 0.15))
+    (fp_line (start 0.35 0.6) (end -0.35 0.6) (layer F.SilkS) (width 0.15))
+    (pad 1 smd rect (at -0.75 0) (size 0.8 0.75) (layers F.Cu F.Paste F.Mask)
+      (net 4 +5V))
+    (pad 2 smd rect (at 0.75 0) (size 0.8 0.75) (layers F.Cu F.Paste F.Mask)
+      (net 2 GND))
+    (model Capacitors_SMD.3dshapes/C_0603.wrl
+      (at (xyz 0 0 0))
+      (scale (xyz 1 1 1))
+      (rotate (xyz 0 0 0))
+    )
+  )
   (module Resistors_SMD:R_0603 (layer B.Cu)
     (at 147.828 116.84)
@@
     )
   )
-  (module open_robotics:DIPSWITCH_SMT_ALCO_2CCT (layer B.Cu)
-    (at 129.667 114.3)
-    (fp_text reference U2 (at 0 3.175) (layer B.SilkS)
-      (effects (font (size 1 1) (thickness 0.15)) (justify mirror))
-    )
-    (fp_text value TE_1825058-1 (at 4.445 1.905) (layer B.Fab)
-      (effects (font (size 1 1) (thickness 0.15)) (justify mirror))
-    )
-    (fp_line (start 10.16 2.54) (end -1.905 2.54) (layer B.CrtYd) (width 0.15))
-    (fp_line (start 10.16 -5.08) (end 10.16 2.54) (layer B.CrtYd) (width 0.15))
-    (fp_line (start -1.905 -5.08) (end 10.16 -5.08) (layer B.CrtYd) (width 0.15))
-    (fp_line (start -1.905 2.54) (end -1.905 -5.08) (layer B.CrtYd) (width 0.15))
-    (pad 1 smd rect (at 0 0) (size 2.159 1.524) (layers B.Cu B.Paste B.Mask)
-      (net 14 /POWER_OUT))
-    (pad 2 smd rect (at 0 -2.54) (size 2.159 1.524) (layers B.Cu B.Paste B.Mask)
-      (net 16 "Net-(J1-Pad7)"))
-    (pad 3 smd rect (at 8.255 -2.54) (size 2.159 1.524) (layers B.Cu B.Paste B.Mask)
-      (net 8 /PROGRAM))
-    (pad 4 smd rect (at 8.255 0) (size 2.159 1.524) (layers B.Cu B.Paste B.Mask)
-      (net 4 +5V))
-  )
   (module Capacitors_SMD:C_0603 (layer F.Cu)
     (at 139.7 118.122 270)
@@
     (pad 1 smd rect (at -0.75 0) (size 0.8 0.75) (layers F.Cu F.Paste F.Mask)
       (net 5 "Net-(C4-Pad1)"))
-    (pad 2 smd rect (at 0.75 0) (size 0.8 0.75) (layers F.Cu F.Paste F.Mask)
-      (net 2 GND))
-    (model Capacitors_SMD.3dshapes/C_0603.wrl
-      (at (xyz 0 0 0))
-      (scale (xyz 1 1 1))
-      (rotate (xyz 0 0 0))
-    )
-  )
-  (module Capacitors_SMD:C_0603 (layer F.Cu)
-    (at 138.696 108.458)
-    (descr "Capacitor SMD 0603, reflow soldering, AVX (see smccp.pdf)")
-    (tags "capacitor 0603")
-    (attr smd)
-    (fp_text reference C5 (at 0 -1.9) (layer F.SilkS)
-      (effects (font (size 1 1) (thickness 0.15)))
-    )
-    (fp_text value 0.1uF (at 0 1.9) (layer F.Fab)
-      (effects (font (size 1 1) (thickness 0.15)))
-    )
-    (fp_line (start -1.45 -0.75) (end 1.45 -0.75) (layer F.CrtYd) (width 0.05))
-    (fp_line (start -1.45 0.75) (end 1.45 0.75) (layer F.CrtYd) (width 0.05))
-    (fp_line (start -1.45 -0.75) (end -1.45 0.75) (layer F.CrtYd) (width 0.05))
-    (fp_line (start 1.45 -0.75) (end 1.45 0.75) (layer F.CrtYd) (width 0.05))
-    (fp_line (start -0.35 -0.6) (end 0.35 -0.6) (layer F.SilkS) (width 0.15))
-    (fp_line (start 0.35 0.6) (end -0.35 0.6) (layer F.SilkS) (width 0.15))
-    (pad 1 smd rect (at -0.75 0) (size 0.8 0.75) (layers F.Cu F.Paste F.Mask)
-      (net 4 +5V))
     (pad 2 smd rect (at 0.75 0) (size 0.8 0.75) (layers F.Cu F.Paste F.Mask)
       (net 2 GND))
@@
       (rotate (xyz 0 0 0))
     )
-  )
-  (module open_robotics:modular8_rev3_edge (layer F.Cu)
-    (at 151.638 112.776 270)
-    (fp_text reference J1 (at -3.81 -3.81 270) (layer F.SilkS) hide
-      (effects (font (size 1 1) (thickness 0.15)))
-    )
-    (fp_text value modular8_rev3_comms_out (at 1.27 -2.54 270) (layer F.Fab) hide
-      (effects (font (size 1 1) (thickness 0.15)))
-    )
-    (pad 1 smd rect (at -5.08 0 270) (size 1.524 2.54) (layers F.Cu F.Paste F.Mask)
-      (net 14 /POWER_OUT))
-    (pad 3 smd rect (at -2.54 0 270) (size 1.524 2.54) (layers F.Cu F.Paste F.Mask)
-      (net 15 "Net-(J1-Pad3)"))
-    (pad 5 smd rect (at 0 0 270) (size 1.524 2.54) (layers F.Cu F.Paste F.Mask)
-      (net 2 GND))
-    (pad 7 smd rect (at 2.54 0 270) (size 1.524 2.54) (layers F.Cu F.Paste F.Mask)
-      (net 16 "Net-(J1-Pad7)"))
-    (pad 9 smd rect (at 5.08 0 270) (size 1.524 2.54) (layers F.Cu F.Paste F.Mask)
-      (net 17 "Net-(J1-Pad9)"))
-    (pad 11 smd rect (at 7.62 0 270) (size 1.524 2.54) (layers F.Cu F.Paste F.Mask)
-      (net 18 "Net-(J1-Pad11)"))
-    (pad 2 smd rect (at -5.08 0 270) (size 1.524 2.54) (layers B.Cu F.Paste F.Mask)
-      (net 19 "Net-(J1-Pad2)"))
-    (pad 4 smd rect (at -2.54 0 270) (size 1.524 2.54) (layers B.Cu F.Paste F.Mask)
-      (net 20 /TX))
-    (pad 6 smd rect (at 0 0 270) (size 1.524 2.54) (layers B.Cu F.Paste F.Mask)
-      (net 21 /RX))
-    (pad 8 smd rect (at 2.54 0 270) (size 1.524 2.54) (layers B.Cu F.Paste F.Mask)
-      (net 2 GND))
-    (pad 10 smd rect (at 5.08 0 270) (size 1.524 2.54) (layers B.Cu F.Paste F.Mask)
-      (net 22 "Net-(J1-Pad10)"))
-    (pad 12 smd rect (at 7.62 0 270) (size 1.524 2.54) (layers B.Cu F.Paste F.Mask)
-      (net 14 /POWER_OUT))
   )
   (module Resistors_SMD:R_0603 (layer F.Cu)
@@
     )
   )
+  (module open_robotics:modular8_rev3_edge (layer F.Cu)
+    (at 151.638 112.776 270)
+    (fp_text reference J1 (at -3.81 -3.81 270) (layer F.SilkS) hide
+      (effects (font (size 1 1) (thickness 0.15)))
+    )
+    (fp_text value modular8_rev3_comms_out (at 1.27 -2.54 270) (layer F.Fab) hide
+      (effects (font (size 1 1) (thickness 0.15)))
+    )
+    (pad 1 smd rect (at -5.08 0 270) (size 1.524 2.54) (layers F.Cu F.Paste F.Mask)
+      (net 14 /POWER_OUT))
+    (pad 3 smd rect (at -2.54 0 270) (size 1.524 2.54) (layers F.Cu F.Paste F.Mask)
+      (net 15 "Net-(J1-Pad3)"))
+    (pad 5 smd rect (at 0 0 270) (size 1.524 2.54) (layers F.Cu F.Paste F.Mask)
+      (net 2 GND))
+    (pad 7 smd rect (at 2.54 0 270) (size 1.524 2.54) (layers F.Cu F.Paste F.Mask)
+      (net 16 "Net-(J1-Pad7)"))
+    (pad 9 smd rect (at 5.08 0 270) (size 1.524 2.54) (layers F.Cu F.Paste F.Mask)
+      (net 17 "Net-(J1-Pad9)"))
+    (pad 11 smd rect (at 7.62 0 270) (size 1.524 2.54) (layers F.Cu F.Paste F.Mask)
+      (net 18 "Net-(J1-Pad11)"))
+    (pad 2 smd rect (at -5.08 0 270) (size 1.524 2.54) (layers B.Cu B.Paste B.Mask)
+      (net 19 "Net-(J1-Pad2)"))
+    (pad 4 smd rect (at -2.54 0 270) (size 1.524 2.54) (layers B.Cu B.Paste B.Mask)
+      (net 20 /TX))
+    (pad 6 smd rect (at 0 0 270) (size 1.524 2.54) (layers B.Cu B.Paste B.Mask)
+      (net 21 /RX))
+    (pad 8 smd rect (at 2.54 0 270) (size 1.524 2.54) (layers B.Cu B.Paste B.Mask)
+      (net 2 GND))
+    (pad 10 smd rect (at 5.08 0 270) (size 1.524 2.54) (layers B.Cu B.Paste B.Mask)
+      (net 22 "Net-(J1-Pad10)"))
+    (pad 12 smd rect (at 7.62 0 270) (size 1.524 2.54) (layers B.Cu B.Paste B.Mask)
+      (net 14 /POWER_OUT))
+  )
+  (gr_text "USB to serial\nChris\nOpenRobotics.ca" (at 127.762 108.966 180) (layer B.SilkS)
+    (effects (font (size 1 1) (thickness 0.1)) (justify left mirror))
+  )
   (gr_line (start 154.178 106.172) (end 127 106.172) (angle 90) (layer Edge.Cuts) (width 0.15))
